File: HW/load-001.sch (KiCad schematic (older format))
At the start: 18 parts

Commit message: Finished hardware design and 3D design
Parts:
- removed RV?: POT_TRIM, symbol POT_TRIM
- added C4: 1nF, Capacitors_ThroughHole:C_Rect_L4_W2.5_P2.5, symbol C_Small
- added J2: Load, suf_connector_ncw:CONN_NCW396-02S, symbol CONN_01X02
- added J3: Range, suf_connector_ncw:CONN_NCW254-03S, symbol CONN_01X03
- added J4: PWR_LED, Pin_Headers:Pin_Header_Straight_1x02, symbol CONN_01X02
- added R2: 47, Resistors_ThroughHole:Resistor_Horizontal_RM10mm, symbol R_Small
- added R6: 100K, Resistors_ThroughHole:Resistor_Horizontal_RM10mm, symbol R_Small
- added R7: 1K, Resistors_ThroughHole:Resistor_Horizontal_RM10mm, symbol R_Small
- added RV4: 50K, Potentiometers:Potentiometer_Bourns_3296W_3-8Zoll_Inline_ScrewUp, symbol POT_TRIM
- C1: renamed from C?; value CP1_Small -> 100uF/35V; footprint (none) -> Capacitors_ThroughHole:C_Radial_D12.5_L25_P5
- C2, C3: renamed from C?; value CP1_Small -> 100uF/16V; footprint (none) -> Capacitors_ThroughHole:C_Radial_D5_L6_P2.5
- D1: renamed from D?; value BRIDGE_1 -> DB106; footprint (none) -> suf_diode_bridge:DB-4
- D2: renamed from D?; value D_Small -> 1N4148; footprint (none) -> Diodes_ThroughHole:Diode_DO-35_SOD27_Horizontal_RM10
- D3: renamed from D?; value ZENERsmall -> BZX55C2V4; footprint (none) -> Diodes_ThroughHole:Diode_DO-35_SOD27_Horizontal_RM10
- J1: renamed from P?; value CONN_01X02 -> AC IN; footprint (none) -> suf_connector_ncw:CONN_NCW254-02S
- Q1: renamed from Q?; value Q_NMOS_GDS -> PHP27NQ11T; footprint (none) -> TO_SOT_Packages_THT:TO-220_Neutral123_Vertical_LargePads
- R1: renamed from R?; value R_Small -> 5.6K; footprint (none) -> Resistors_ThroughHole:Resistor_Horizontal_RM10mm
- R3: renamed from R?; value R_Small -> 1K; footprint (none) -> Resistors_ThroughHole:Resistor_Horizontal_RM10mm
- R4: renamed from R?; value R_Small -> 100; footprint (none) -> Resistors_ThroughHole:Resistor_Horizontal_RM10mm
- R5: renamed from R?; value R_Small -> 1; footprint (none) -> Resistors_ThroughHole:Resistor_Horizontal_RM25mm
- RV1: renamed from RV?; value POT_TRIM -> 50; footprint (none) -> Potentiometers:Potentiometer_Bourns_3296W_3-8Zoll_Inline_ScrewUp
- RV2: renamed from RV?; value POT_TRIM -> 10K; footprint (none) -> Potentiometers:Potentiometer_Bourns_3296W_3-8Zoll_Inline_ScrewUp
- RV3: renamed from RV?; value POT -> 10K; footprint (none) -> suf_connector_ncw:CONN_NCW254-03S
- U1: renamed from U?; footprint (none) -> TO_SOT_Packages_THT:TO-220_Neutral123_Vertical_LargePads
- U2: renamed from U?; value LM358 -> TS358; footprint (none) -> Housings_DIP:DIP-8_W7.62mm_LongPads
Connections:
- net GND: now also R5.2, C4.2, J2.2 (P2), J4.2 (P2)
- net VCC: now also U2.8 (V+), R7.1
- net at C1.2, C3.2, D1.1 (-)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: now also R2.2; no longer RV1.3
- net at D3.1 (K), R3.2, RV2.1: now also R6.1
- net at RV2.2, RV2.3: now also J3.3 (P3); no longer RV3.1
- net at RV3.2, U2.3 (+): now also C4.1
- net at Q1.2 (D): now also J2.1 (P1)
- new net: R2.1, RV1.3
- new net: J3.2 (P2), RV3.1
- new net: R6.2, RV4.1
- new net: J3.1 (P1), RV4.2, RV4.3
- new net: J4.1 (P1), R7.2
Other:
- moved on the sheet: C1, C2, C3, D2, D3, R1, R3, RV1, RV2, RV3, U1
